Commit message: Fix URDF world frame

File: ROS2/ros2_scara_ws/src/dalsa_bioscara/bioscara_description/urdf/bioscara.urdf.xacro (robot description, xacro)
@@ -1,4 +1,5 @@
 <?xml version="1.0" ?>
 <robot xmlns:xacro="http://www.ros.org/wiki/xacro">
+<link name="world" />
 <link name="base_link">
   <inertial>
@@ -101,4 +102,9 @@
   </collision>
 </link>
+<joint name="base_joint" type="fixed">
+  <origin xyz="0 0 0" rpy="0 0 0" />
+  <parent link="world" />
+  <child link="base_link" />
+</joint>
 <joint name="j1" type="revolute">
   <origin xyz="0.0 0.0 0.1442" rpy="0 0 0"/>
@@ -129,9 +135,9 @@
   <limit upper="2.96706" lower="-2.96706" effort="100" velocity="100"/>
 </joint>
-  <joint name="tool_joint" type="fixed">
-    <origin xyz="0 0 0" rpy="${pi} 0 0" />
-    <parent link="link_4"/>
-    <child link="tool0" />
-  </joint>
+<joint name="tool_joint" type="fixed">
+  <origin xyz="0 0 0" rpy="${pi} 0 0" />
+  <parent link="link_4"/>
+  <child link="tool0" />
+</joint>
   <!-- Tool Link -->
   <link name="tool0">

Commit message: change controller update rate

File: ROS2/ros2_scara_ws/src/dalsa_bioscara/bioscara_description/urdf/bioscara.urdf.xacro (robot description, xacro)
@@ -1,5 +1,6 @@
 <?xml version="1.0" ?>
 <robot xmlns:xacro="http://www.ros.org/wiki/xacro">
-<link name="world" />
+<link name="world">
+</link>
 <link name="base_link">
   <inertial>
@@ -102,4 +103,7 @@
   </collision>
 </link>
+<!-- Tool Link -->
+<link name="tool0">
+</link>
 <joint name="base_joint" type="fixed">
   <origin xyz="0 0 0" rpy="0 0 0" />
@@ -140,6 +144,3 @@
   <child link="tool0" />
 </joint>
-  <!-- Tool Link -->
-  <link name="tool0">
-  </link>
 </robot>

Commit message: test: use params from yaml

File: ROS2/ros2_scara_ws/src/dalsa_bioscara/bioscara_description/urdf/bioscara.urdf.xacro (robot description, xacro)
@@ -1,146 +1,148 @@
 <?xml version="1.0" ?>
 <robot xmlns:xacro="http://www.ros.org/wiki/xacro">
-<link name="world">
-</link>
-<link name="base_link">
-  <inertial>
-    <origin xyz="-0.04726295478480471 -4.0726333219249673e-17 0.039609285941398516" rpy="0 0 0"/>
-    <mass value="42.07322100213777"/>
-    <inertia ixx="0.19661" iyy="0.332522" izz="0.481291" ixy="-0.0" iyz="-0.0" ixz="-0.016821"/>
-  </inertial>
-  <visual>
-    <origin xyz="0 0 0" rpy="0 0 0"/>
-    <geometry>
-      <mesh filename="file://$(find bioscara_description)/meshes/base_link.stl" scale="0.001 0.001 0.001"/>
-    </geometry>
-    <material name="silver"/>
-  </visual>
-  <collision>
-    <origin xyz="0 0 0" rpy="0 0 0"/>
-    <geometry>
-      <mesh filename="file://$(find bioscara_description)/meshes/base_link.stl" scale="0.001 0.001 0.001"/>
-    </geometry>
-  </collision>
-</link>
-<link name="link_1">
-  <inertial>
-    <origin xyz="-0.015985049353244893 0.0 0.22758900000000004" rpy="0 0 0"/>
-    <mass value="201.06235973556932"/>
-    <inertia ixx="6.011699" iyy="6.341964" izz="1.505144" ixy="0.0" iyz="0.0" ixz="0.0"/>
-  </inertial>
-  <visual>
-    <origin xyz="-0.0 -0.0 -0.1442" rpy="0 0 0"/>
-    <geometry>
-      <mesh filename="file://$(find bioscara_description)/meshes/link_1_1.stl" scale="0.001 0.001 0.001"/>
-    </geometry>
-    <material name="silver"/>
-  </visual>
-  <collision>
-    <origin xyz="-0.0 -0.0 -0.1442" rpy="0 0 0"/>
-    <geometry>
-      <mesh filename="file://$(find bioscara_description)/meshes/link_1_1.stl" scale="0.001 0.001 0.001"/>
-    </geometry>
-  </collision>
-</link>
-<link name="link_2">
-  <inertial>
-    <origin xyz="0.16393794060138223 0.0 0.06413863377953821" rpy="0 0 0"/>
-    <mass value="31.7907164853462"/>
-    <inertia ixx="0.067297" iyy="0.418803" izz="0.409122" ixy="-0.0" iyz="0.0" ixz="-0.039463"/>
-  </inertial>
-  <visual>
-    <origin xyz="-0.0 -0.0 -0.1442" rpy="0 0 0"/>
-    <geometry>
-      <mesh filename="file://$(find bioscara_description)/meshes/link_2_1.stl" scale="0.001 0.001 0.001"/>
-    </geometry>
-    <material name="silver"/>
-  </visual>
-  <collision>
-    <origin xyz="-0.0 -0.0 -0.1442" rpy="0 0 0"/>
-    <geometry>
-      <mesh filename="file://$(find bioscara_description)/meshes/link_2_1.stl" scale="0.001 0.001 0.001"/>
-    </geometry>
-  </collision>
-</link>
-<link name="link_3">
-  <inertial>
-    <origin xyz="0.14250000161157844 -4.518384865479846e-17 0.08014650000000001" rpy="0 0 0"/>
-    <mass value="28.44193338693538"/>
-    <inertia ixx="0.063431" iyy="0.329798" izz="0.289827" ixy="-0.0" iyz="-0.0" ixz="0.0"/>
-  </inertial>
-  <visual>
-    <origin xyz="-0.329476 -0.0 -0.1442" rpy="0 0 0"/>
-    <geometry>
-      <mesh filename="file://$(find bioscara_description)/meshes/link_3_1.stl" scale="0.001 0.001 0.001"/>
-    </geometry>
-    <material name="silver"/>
-  </visual>
-  <collision>
-    <origin xyz="-0.329476 -0.0 -0.1442" rpy="0 0 0"/>
-    <geometry>
-      <mesh filename="file://$(find bioscara_description)/meshes/link_3_1.stl" scale="0.001 0.001 0.001"/>
-    </geometry>
-  </collision>
-</link>
-<link name="link_4">
-  <inertial>
-    <origin xyz="3.2231565194607015e-09 -4.5766223964710255e-17 0.06973284751916564" rpy="0 0 0"/>
-    <mass value="1.4470826717389633"/>
-    <inertia ixx="0.002924" iyy="0.003053" izz="0.000318" ixy="0.0" iyz="0.0" ixz="-0.0"/>
-  </inertial>
-  <visual>
-    <origin xyz="-0.614476 0.0 -0.1442" rpy="0 0 0"/>
-    <geometry>
-      <mesh filename="file://$(find bioscara_description)/meshes/link_4_1.stl" scale="0.001 0.001 0.001"/>
-    </geometry>
-    <material name="silver"/>
-  </visual>
-  <collision>
-    <origin xyz="-0.614476 0.0 -0.1442" rpy="0 0 0"/>
-    <geometry>
-      <mesh filename="file://$(find bioscara_description)/meshes/link_4_1.stl" scale="0.001 0.001 0.001"/>
-    </geometry>
-  </collision>
-</link>
-<!-- Tool Link -->
-<link name="tool0">
-</link>
-<joint name="base_joint" type="fixed">
-  <origin xyz="0 0 0" rpy="0 0 0" />
-  <parent link="world" />
-  <child link="base_link" />
-</joint>
-<joint name="j1" type="revolute">
-  <origin xyz="0.0 0.0 0.1442" rpy="0 0 0"/>
-  <parent link="base_link"/>
-  <child link="link_1"/>
-  <axis xyz="0.0 0.0 1.0"/>
-  <limit upper="2.96706" lower="-2.96706" effort="100" velocity="100"/>
-</joint>
-<joint name="j2" type="prismatic">
-  <origin xyz="0.0 0.0 0.0" rpy="0 0 0"/>
-  <parent link="link_1"/>
-  <child link="link_2"/>
-  <axis xyz="0.0 0.0 1.0"/>
-  <limit upper="0.338" lower="0.0" effort="100" velocity="100"/>
-</joint>
-<joint name="j3" type="revolute">
-  <origin xyz="0.329476 0.0 0.0" rpy="0 0 0"/>
-  <parent link="link_2"/>
-  <child link="link_3"/>
-  <axis xyz="0.0 0.0 1.0"/>
-  <limit upper="2.96706" lower="-2.96706" effort="100" velocity="100"/>
-</joint>
-<joint name="j4" type="revolute">
-  <origin xyz="0.285 -0.0 0.0" rpy="0 0 0"/>
-  <parent link="link_3"/>
-  <child link="link_4"/>
-  <axis xyz="0.0 0.0 1.0"/>
-  <limit upper="2.96706" lower="-2.96706" effort="100" velocity="100"/>
-</joint>
-<joint name="tool_joint" type="fixed">
-  <origin xyz="0 0 0" rpy="${pi} 0 0" />
-  <parent link="link_4"/>
-  <child link="tool0" />
-</joint>
+  <xacro:property name="config_file" value="$(find bioscara_description)/config/bioscara_parameters.yaml" />
+  <xacro:property name="params" value="${load_yaml(config_file)}"/>
+  <link name="world">
+  </link>
+  <link name="base_link">
+    <inertial>
+      <origin xyz="-0.04726295478480471 -4.0726333219249673e-17 0.039609285941398516" rpy="0 0 0"/>
+      <mass value="42.07322100213777"/>
+      <inertia ixx="0.19661" iyy="0.332522" izz="0.481291" ixy="-0.0" iyz="-0.0" ixz="-0.016821"/>
+    </inertial>
+    <visual>
+      <origin xyz="0 0 0" rpy="0 0 0"/>
+      <geometry>
+        <mesh filename="file://$(find bioscara_description)/meshes/base_link.stl" scale="0.001 0.001 0.001"/>
+      </geometry>
+      <material name="silver"/>
+    </visual>
+    <collision>
+      <origin xyz="0 0 0" rpy="0 0 0"/>
+      <geometry>
+        <mesh filename="file://$(find bioscara_description)/meshes/base_link.stl" scale="0.001 0.001 0.001"/>
+      </geometry>
+    </collision>
+  </link>
+  <link name="link_1">
+    <inertial>
+      <origin xyz="-0.015985049353244893 0.0 0.22758900000000004" rpy="0 0 0"/>
+      <mass value="201.06235973556932"/>
+      <inertia ixx="6.011699" iyy="6.341964" izz="1.505144" ixy="0.0" iyz="0.0" ixz="0.0"/>
+    </inertial>
+    <visual>
+      <origin xyz="-0.0 -0.0 -0.1442" rpy="0 0 0"/>
+      <geometry>
+        <mesh filename="file://$(find bioscara_description)/meshes/link_1_1.stl" scale="0.001 0.001 0.001"/>
+      </geometry>
+      <material name="silver"/>
+    </visual>
+    <collision>
+      <origin xyz="-0.0 -0.0 -0.1442" rpy="0 0 0"/>
+      <geometry>
+        <mesh filename="file://$(find bioscara_description)/meshes/link_1_1.stl" scale="0.001 0.001 0.001"/>
+      </geometry>
+    </collision>
+  </link>
+  <link name="link_2">
+    <inertial>
+      <origin xyz="0.16393794060138223 0.0 0.06413863377953821" rpy="0 0 0"/>
+      <mass value="31.7907164853462"/>
+      <inertia ixx="0.067297" iyy="0.418803" izz="0.409122" ixy="-0.0" iyz="0.0" ixz="-0.039463"/>
+    </inertial>
+    <visual>
+      <origin xyz="-0.0 -0.0 -0.1442" rpy="0 0 0"/>
+      <geometry>
+        <mesh filename="file://$(find bioscara_description)/meshes/link_2_1.stl" scale="0.001 0.001 0.001"/>
+      </geometry>
+      <material name="silver"/>
+    </visual>
+    <collision>
+      <origin xyz="-0.0 -0.0 -0.1442" rpy="0 0 0"/>
+      <geometry>
+        <mesh filename="file://$(find bioscara_description)/meshes/link_2_1.stl" scale="0.001 0.001 0.001"/>
+      </geometry>
+    </collision>
+  </link>
+  <link name="link_3">
+    <inertial>
+      <origin xyz="0.14250000161157844 -4.518384865479846e-17 0.08014650000000001" rpy="0 0 0"/>
+      <mass value="28.44193338693538"/>
+      <inertia ixx="0.063431" iyy="0.329798" izz="0.289827" ixy="-0.0" iyz="-0.0" ixz="0.0"/>
+    </inertial>
+    <visual>
+      <origin xyz="-0.329476 -0.0 -0.1442" rpy="0 0 0"/>
+      <geometry>
+        <mesh filename="file://$(find bioscara_description)/meshes/link_3_1.stl" scale="0.001 0.001 0.001"/>
+      </geometry>
+      <material name="silver"/>
+    </visual>
+    <collision>
+      <origin xyz="-0.329476 -0.0 -0.1442" rpy="0 0 0"/>
+      <geometry>
+        <mesh filename="file://$(find bioscara_description)/meshes/link_3_1.stl" scale="0.001 0.001 0.001"/>
+      </geometry>
+    </collision>
+  </link>
+  <link name="link_4">
+    <inertial>
+      <origin xyz="3.2231565194607015e-09 -4.5766223964710255e-17 0.06973284751916564" rpy="0 0 0"/>
+      <mass value="1.4470826717389633"/>
+      <inertia ixx="0.002924" iyy="0.003053" izz="0.000318" ixy="0.0" iyz="0.0" ixz="-0.0"/>
+    </inertial>
+    <visual>
+      <origin xyz="-0.614476 0.0 -0.1442" rpy="0 0 0"/>
+      <geometry>
+        <mesh filename="file://$(find bioscara_description)/meshes/link_4_1.stl" scale="0.001 0.001 0.001"/>
+      </geometry>
+      <material name="silver"/>
+    </visual>
+    <collision>
+      <origin xyz="-0.614476 0.0 -0.1442" rpy="0 0 0"/>
+      <geometry>
+        <mesh filename="file://$(find bioscara_description)/meshes/link_4_1.stl" scale="0.001 0.001 0.001"/>
+      </geometry>
+    </collision>
+  </link>
+  <!-- Tool Link -->
+  <link name="tool0">
+  </link>
+  <joint name="base_joint" type="fixed">
+    <origin xyz="0 0 0" rpy="0 0 0" />
+    <parent link="world" />
+    <child link="base_link" />
+  </joint>
+  <joint name="j1" type="revolute">
+    <origin xyz="0.0 0.0 0.1442" rpy="0 0 0"/>
+    <parent link="base_link"/>
+    <child link="link_1"/>
+    <axis xyz="0.0 0.0 1.0"/>
+    <limit upper="${abs(params['j1']['offset']}" lower="${0-abs(params['j1']['offset']}" effort="100" velocity="100"/>
+  </joint>
+  <joint name="j2" type="prismatic">
+    <origin xyz="0.0 0.0 0.0" rpy="0 0 0"/>
+    <parent link="link_1"/>
+    <child link="link_2"/>
+    <axis xyz="0.0 0.0 1.0"/>
+    <limit upper="0.338" lower="0.0" effort="100" velocity="100"/>
+  </joint>
+  <joint name="j3" type="revolute">
+    <origin xyz="0.329476 0.0 0.0" rpy="0 0 0"/>
+    <parent link="link_2"/>
+    <child link="link_3"/>
+    <axis xyz="0.0 0.0 1.0"/>
+    <limit upper="2.96706" lower="-2.96706" effort="100" velocity="100"/>
+  </joint>
+  <joint name="j4" type="revolute">
+    <origin xyz="0.285 -0.0 0.0" rpy="0 0 0"/>
+    <parent link="link_3"/>
+    <child link="link_4"/>
+    <axis xyz="0.0 0.0 1.0"/>
+    <limit upper="2.96706" lower="-2.96706" effort="100" velocity="100"/>
+  </joint>
+  <joint name="tool_joint" type="fixed">
+    <origin xyz="0 0 0" rpy="${pi} 0 0" />
+    <parent link="link_4"/>
+    <child link="tool0" />
+  </joint>
 </robot>

Commit message: config from yaml, urdf part

File: ROS2/ros2_scara_ws/src/dalsa_bioscara/bioscara_description/urdf/bioscara.urdf.xacro (robot description, xacro)
@@ -118,5 +118,5 @@
     <child link="link_1"/>
     <axis xyz="0.0 0.0 1.0"/>
-    <limit upper="${abs(params['j1']['offset']}" lower="${0-abs(params['j1']['offset']}" effort="100" velocity="100"/>
+    <limit upper="${fabs(params['j1']['offset'])}" lower="${0-fabs(params['j1']['offset'])}" effort="100" velocity="${params['j1']['max_velocity']}"/>
   </joint>
   <joint name="j2" type="prismatic">
@@ -125,5 +125,5 @@
     <child link="link_2"/>
     <axis xyz="0.0 0.0 1.0"/>
-    <limit upper="0.338" lower="0.0" effort="100" velocity="100"/>
+    <limit upper="${params['j2']['offset']}" lower="0" effort="100" velocity="${params['j2']['max_velocity']}"/>
   </joint>
   <joint name="j3" type="revolute">
@@ -132,5 +132,5 @@
     <child link="link_3"/>
     <axis xyz="0.0 0.0 1.0"/>
-    <limit upper="2.96706" lower="-2.96706" effort="100" velocity="100"/>
+    <limit upper="${fabs(params['j3']['offset'])}" lower="${0-fabs(params['j3']['offset'])}" effort="100" velocity="${params['j3']['max_velocity']}"/>
   </joint>
   <joint name="j4" type="revolute">
@@ -139,5 +139,5 @@
     <child link="link_4"/>
     <axis xyz="0.0 0.0 1.0"/>
-    <limit upper="2.96706" lower="-2.96706" effort="100" velocity="100"/>
+    <limit upper="${fabs(params['j4']['offset'])}" lower="${0-fabs(params['j4']['offset'])}" effort="100" velocity="${params['j4']['max_velocity']}"/>
   </joint>
   <joint name="tool_joint" type="fixed">

Commit message: fixed parsing issues

File: ROS2/ros2_scara_ws/src/dalsa_bioscara/bioscara_description/urdf/bioscara.urdf.xacro (robot description, xacro)
@@ -2,5 +2,5 @@
 <robot xmlns:xacro="http://www.ros.org/wiki/xacro">
   <xacro:property name="config_file" value="$(find bioscara_description)/config/bioscara_parameters.yaml" />
-  <xacro:property name="params" value="${load_yaml(config_file)}"/>
+  <xacro:property name="params" value="${xacro.load_yaml(config_file)}"/>
   <link name="world">
   </link>
