Commit message: macro-fy description

File: ROS2/ros2_scara_ws/src/dalsa_bioscara/bioscara_description/urdf/bioscara.urdf.xacro (robot description, xacro)
@@ -1,148 +1,145 @@
 <?xml version="1.0" ?>
 <robot xmlns:xacro="http://www.ros.org/wiki/xacro">
-  <xacro:property name="config_file" value="$(find bioscara_description)/config/bioscara_parameters.yaml" />
-  <xacro:property name="params" value="${xacro.load_yaml(config_file)}"/>
-  <link name="world">
-  </link>
-  <link name="base_link">
-    <inertial>
-      <origin xyz="-0.04726295478480471 -4.0726333219249673e-17 0.039609285941398516" rpy="0 0 0"/>
-      <mass value="42.07322100213777"/>
-      <inertia ixx="0.19661" iyy="0.332522" izz="0.481291" ixy="-0.0" iyz="-0.0" ixz="-0.016821"/>
-    </inertial>
-    <visual>
-      <origin xyz="0 0 0" rpy="0 0 0"/>
-      <geometry>
-        <mesh filename="file://$(find bioscara_description)/meshes/base_link.stl" scale="0.001 0.001 0.001"/>
-      </geometry>
-      <material name="silver"/>
-    </visual>
-    <collision>
-      <origin xyz="0 0 0" rpy="0 0 0"/>
-      <geometry>
-        <mesh filename="file://$(find bioscara_description)/meshes/base_link.stl" scale="0.001 0.001 0.001"/>
-      </geometry>
-    </collision>
-  </link>
-  <link name="link_1">
-    <inertial>
-      <origin xyz="-0.015985049353244893 0.0 0.22758900000000004" rpy="0 0 0"/>
-      <mass value="201.06235973556932"/>
-      <inertia ixx="6.011699" iyy="6.341964" izz="1.505144" ixy="0.0" iyz="0.0" ixz="0.0"/>
-    </inertial>
-    <visual>
-      <origin xyz="-0.0 -0.0 -0.1442" rpy="0 0 0"/>
-      <geometry>
-        <mesh filename="file://$(find bioscara_description)/meshes/link_1_1.stl" scale="0.001 0.001 0.001"/>
-      </geometry>
-      <material name="silver"/>
-    </visual>
-    <collision>
-      <origin xyz="-0.0 -0.0 -0.1442" rpy="0 0 0"/>
-      <geometry>
-        <mesh filename="file://$(find bioscara_description)/meshes/link_1_1.stl" scale="0.001 0.001 0.001"/>
-      </geometry>
-    </collision>
-  </link>
-  <link name="link_2">
-    <inertial>
-      <origin xyz="0.16393794060138223 0.0 0.06413863377953821" rpy="0 0 0"/>
-      <mass value="31.7907164853462"/>
-      <inertia ixx="0.067297" iyy="0.418803" izz="0.409122" ixy="-0.0" iyz="0.0" ixz="-0.039463"/>
-    </inertial>
-    <visual>
-      <origin xyz="-0.0 -0.0 -0.1442" rpy="0 0 0"/>
-      <geometry>
-        <mesh filename="file://$(find bioscara_description)/meshes/link_2_1.stl" scale="0.001 0.001 0.001"/>
-      </geometry>
-      <material name="silver"/>
-    </visual>
-    <collision>
-      <origin xyz="-0.0 -0.0 -0.1442" rpy="0 0 0"/>
-      <geometry>
-        <mesh filename="file://$(find bioscara_description)/meshes/link_2_1.stl" scale="0.001 0.001 0.001"/>
-      </geometry>
-    </collision>
-  </link>
-  <link name="link_3">
-    <inertial>
-      <origin xyz="0.14250000161157844 -4.518384865479846e-17 0.08014650000000001" rpy="0 0 0"/>
-      <mass value="28.44193338693538"/>
-      <inertia ixx="0.063431" iyy="0.329798" izz="0.289827" ixy="-0.0" iyz="-0.0" ixz="0.0"/>
-    </inertial>
-    <visual>
-      <origin xyz="-0.329476 -0.0 -0.1442" rpy="0 0 0"/>
-      <geometry>
-        <mesh filename="file://$(find bioscara_description)/meshes/link_3_1.stl" scale="0.001 0.001 0.001"/>
-      </geometry>
-      <material name="silver"/>
-    </visual>
-    <collision>
-      <origin xyz="-0.329476 -0.0 -0.1442" rpy="0 0 0"/>
-      <geometry>
-        <mesh filename="file://$(find bioscara_description)/meshes/link_3_1.stl" scale="0.001 0.001 0.001"/>
-      </geometry>
-    </collision>
-  </link>
-  <link name="link_4">
-    <inertial>
-      <origin xyz="3.2231565194607015e-09 -4.5766223964710255e-17 0.06973284751916564" rpy="0 0 0"/>
-      <mass value="1.4470826717389633"/>
-      <inertia ixx="0.002924" iyy="0.003053" izz="0.000318" ixy="0.0" iyz="0.0" ixz="-0.0"/>
-    </inertial>
-    <visual>
-      <origin xyz="-0.614476 0.0 -0.1442" rpy="0 0 0"/>
-      <geometry>
-        <mesh filename="file://$(find bioscara_description)/meshes/link_4_1.stl" scale="0.001 0.001 0.001"/>
-      </geometry>
-      <material name="silver"/>
-    </visual>
-    <collision>
-      <origin xyz="-0.614476 0.0 -0.1442" rpy="0 0 0"/>
-      <geometry>
-        <mesh filename="file://$(find bioscara_description)/meshes/link_4_1.stl" scale="0.001 0.001 0.001"/>
-      </geometry>
-    </collision>
-  </link>
-  <!-- Tool Link -->
-  <link name="tool0">
-  </link>
-  <joint name="base_joint" type="fixed">
-    <origin xyz="0 0 0" rpy="0 0 0" />
-    <parent link="world" />
-    <child link="base_link" />
-  </joint>
-  <joint name="j1" type="revolute">
-    <origin xyz="0.0 0.0 0.1442" rpy="0 0 0"/>
-    <parent link="base_link"/>
-    <child link="link_1"/>
-    <axis xyz="0.0 0.0 1.0"/>
-    <limit upper="${fabs(params['j1']['offset'])}" lower="${0-fabs(params['j1']['offset'])}" effort="100" velocity="${params['j1']['max_velocity']}"/>
-  </joint>
-  <joint name="j2" type="prismatic">
-    <origin xyz="0.0 0.0 0.0" rpy="0 0 0"/>
-    <parent link="link_1"/>
-    <child link="link_2"/>
-    <axis xyz="0.0 0.0 1.0"/>
-    <limit upper="${params['j2']['offset']}" lower="0" effort="100" velocity="${params['j2']['max_velocity']}"/>
-  </joint>
-  <joint name="j3" type="revolute">
-    <origin xyz="0.329476 0.0 0.0" rpy="0 0 0"/>
-    <parent link="link_2"/>
-    <child link="link_3"/>
-    <axis xyz="0.0 0.0 1.0"/>
-    <limit upper="${fabs(params['j3']['offset'])}" lower="${0-fabs(params['j3']['offset'])}" effort="100" velocity="${params['j3']['max_velocity']}"/>
-  </joint>
-  <joint name="j4" type="revolute">
-    <origin xyz="0.285 -0.0 0.0" rpy="0 0 0"/>
-    <parent link="link_3"/>
-    <child link="link_4"/>
-    <axis xyz="0.0 0.0 1.0"/>
-    <limit upper="${fabs(params['j4']['offset'])}" lower="${0-fabs(params['j4']['offset'])}" effort="100" velocity="${params['j4']['max_velocity']}"/>
-  </joint>
-  <joint name="tool_joint" type="fixed">
-    <origin xyz="0 0 0" rpy="${pi} 0 0" />
-    <parent link="link_4"/>
-    <child link="tool0" />
-  </joint>
+  <xacro:macro name="bioscara" params="parameters prefix parent *origin">
+    <joint name="${prefix}base_joint" type="fixed">
+      <xacro:insert_block name="origin" />
+      <parent link="${parent}" />
+      <child link="${prefix}base_link" />
+    </joint>
+    <link name="${prefix}base_link">
+      <inertial>
+        <origin xyz="-0.04726295478480471 -4.0726333219249673e-17 0.039609285941398516" rpy="0 0 0"/>
+        <mass value="42.07322100213777"/>
+        <inertia ixx="0.19661" iyy="0.332522" izz="0.481291" ixy="-0.0" iyz="-0.0" ixz="-0.016821"/>
+      </inertial>
+      <visual>
+        <origin xyz="0 0 0" rpy="0 0 0"/>
+        <geometry>
+          <mesh filename="file://$(find bioscara_description)/meshes/base_link.stl" scale="0.001 0.001 0.001"/>
+        </geometry>
+        <material name="silver"/>
+      </visual>
+      <collision>
+        <origin xyz="0 0 0" rpy="0 0 0"/>
+        <geometry>
+          <mesh filename="file://$(find bioscara_description)/meshes/base_link.stl" scale="0.001 0.001 0.001"/>
+        </geometry>
+      </collision>
+    </link>
+    <joint name="${prefix}j1" type="revolute">
+      <origin xyz="0.0 0.0 0.1442" rpy="0 0 0"/>
+      <parent link="${prefix}base_link"/>
+      <child link="${prefix}link_1"/>
+      <axis xyz="0.0 0.0 1.0"/>
+      <limit upper="${fabs(parameters['j1']['offset'])}" lower="${0-fabs(parameters['j1']['offset'])}" effort="100" velocity="${parameters['j1']['max_velocity']}"/>
+    </joint>
+    <link name="${prefix}link_1">
+      <inertial>
+        <origin xyz="-0.015985049353244893 0.0 0.22758900000000004" rpy="0 0 0"/>
+        <mass value="201.06235973556932"/>
+        <inertia ixx="6.011699" iyy="6.341964" izz="1.505144" ixy="0.0" iyz="0.0" ixz="0.0"/>
+      </inertial>
+      <visual>
+        <origin xyz="-0.0 -0.0 -0.1442" rpy="0 0 0"/>
+        <geometry>
+          <mesh filename="file://$(find bioscara_description)/meshes/link_1_1.stl" scale="0.001 0.001 0.001"/>
+        </geometry>
+        <material name="silver"/>
+      </visual>
+      <collision>
+        <origin xyz="-0.0 -0.0 -0.1442" rpy="0 0 0"/>
+        <geometry>
+          <mesh filename="file://$(find bioscara_description)/meshes/link_1_1.stl" scale="0.001 0.001 0.001"/>
+        </geometry>
+      </collision>
+    </link>
+    <joint name="${prefix}j2" type="prismatic">
+      <origin xyz="0.0 0.0 0.0" rpy="0 0 0"/>
+      <parent link="${prefix}link_1"/>
+      <child link="${prefix}link_2"/>
+      <axis xyz="0.0 0.0 1.0"/>
+      <limit upper="${parameters['j2']['offset']}" lower="0" effort="100" velocity="${parameters['j2']['max_velocity']}"/>
+    </joint>
+    <link name="${prefix}link_2">
+      <inertial>
+        <origin xyz="0.16393794060138223 0.0 0.06413863377953821" rpy="0 0 0"/>
+        <mass value="31.7907164853462"/>
+        <inertia ixx="0.067297" iyy="0.418803" izz="0.409122" ixy="-0.0" iyz="0.0" ixz="-0.039463"/>
+      </inertial>
+      <visual>
+        <origin xyz="-0.0 -0.0 -0.1442" rpy="0 0 0"/>
+        <geometry>
+          <mesh filename="file://$(find bioscara_description)/meshes/link_2_1.stl" scale="0.001 0.001 0.001"/>
+        </geometry>
+        <material name="silver"/>
+      </visual>
+      <collision>
+        <origin xyz="-0.0 -0.0 -0.1442" rpy="0 0 0"/>
+        <geometry>
+          <mesh filename="file://$(find bioscara_description)/meshes/link_2_1.stl" scale="0.001 0.001 0.001"/>
+        </geometry>
+      </collision>
+    </link>
+    <joint name="${prefix}j3" type="revolute">
+      <origin xyz="0.329476 0.0 0.0" rpy="0 0 0"/>
+      <parent link="${prefix}link_2"/>
+      <child link="${prefix}link_3"/>
+      <axis xyz="0.0 0.0 1.0"/>
+      <limit upper="${fabs(parameters['j3']['offset'])}" lower="${0-fabs(parameters['j3']['offset'])}" effort="100" velocity="${parameters['j3']['max_velocity']}"/>
+    </joint>
+    <link name="${prefix}link_3">
+      <inertial>
+        <origin xyz="0.14250000161157844 -4.518384865479846e-17 0.08014650000000001" rpy="0 0 0"/>
+        <mass value="28.44193338693538"/>
+        <inertia ixx="0.063431" iyy="0.329798" izz="0.289827" ixy="-0.0" iyz="-0.0" ixz="0.0"/>
+      </inertial>
+      <visual>
+        <origin xyz="-0.329476 -0.0 -0.1442" rpy="0 0 0"/>
+        <geometry>
+          <mesh filename="file://$(find bioscara_description)/meshes/link_3_1.stl" scale="0.001 0.001 0.001"/>
+        </geometry>
+        <material name="silver"/>
+      </visual>
+      <collision>
+        <origin xyz="-0.329476 -0.0 -0.1442" rpy="0 0 0"/>
+        <geometry>
+          <mesh filename="file://$(find bioscara_description)/meshes/link_3_1.stl" scale="0.001 0.001 0.001"/>
+        </geometry>
+      </collision>
+    </link>
+    <joint name="${prefix}j4" type="revolute">
+      <origin xyz="0.285 -0.0 0.0" rpy="0 0 0"/>
+      <parent link="${prefix}link_3"/>
+      <child link="${prefix}link_4"/>
+      <axis xyz="0.0 0.0 1.0"/>
+      <limit upper="${fabs(parameters['j4']['offset'])}" lower="${0-fabs(parameters['j4']['offset'])}" effort="100" velocity="${parameters['j4']['max_velocity']}"/>
+    </joint>
+    <link name="${prefix}link_4">
+      <inertial>
+        <origin xyz="3.2231565194607015e-09 -4.5766223964710255e-17 0.06973284751916564" rpy="0 0 0"/>
+        <mass value="1.4470826717389633"/>
+        <inertia ixx="0.002924" iyy="0.003053" izz="0.000318" ixy="0.0" iyz="0.0" ixz="-0.0"/>
+      </inertial>
+      <visual>
+        <origin xyz="-0.614476 0.0 -0.1442" rpy="0 0 0"/>
+        <geometry>
+          <mesh filename="file://$(find bioscara_description)/meshes/link_4_1.stl" scale="0.001 0.001 0.001"/>
+        </geometry>
+        <material name="silver"/>
+      </visual>
+      <collision>
+        <origin xyz="-0.614476 0.0 -0.1442" rpy="0 0 0"/>
+        <geometry>
+          <mesh filename="file://$(find bioscara_description)/meshes/link_4_1.stl" scale="0.001 0.001 0.001"/>
+        </geometry>
+      </collision>
+    </link>
+    <joint name="${prefix}tool_joint" type="fixed">
+      <origin xyz="0 0 0" rpy="${pi} 0 0" />
+      <parent link="${prefix}link_4"/>
+      <child link="${prefix}tool0" />
+    </joint>
+    <!-- Tool Link -->
+    <link name="${prefix}tool0"/>
+  </xacro:macro>
 </robot>

File: ROS2/ros2_scara_ws/src/dalsa_bioscara/bioscara_description/urdf/bioscara.xacro (robot description, xacro)
@@ -3,12 +3,15 @@
   <xacro:arg name="use_mock_hardware" default="false"/>
   <xacro:arg name="prefix" default=""/>
+  <xacro:property name="config_file" value="$(find bioscara_description)/config/bioscara_parameters.yaml" />
+  <xacro:property name="params" value="${xacro.load_yaml(config_file)}"/>
   <xacro:include filename="$(find bioscara_description)/urdf/materials.xacro" />
-  <xacro:if value="$(arg use_mock_hardware)">
-      <xacro:include filename="$(find bioscara_description)/urdf/bioscara_mock.ros2control" />
-  </xacro:if>
-  <xacro:unless value="$(arg use_mock_hardware)">
-      <xacro:include filename="$(find bioscara_description)/urdf/bioscara.ros2control" />
-  </xacro:unless>
+  <xacro:include filename="$(find bioscara_description)/urdf/bioscara.urdf.xacro" />
   <xacro:include filename="$(find bioscara_description)/urdf/bioscara.gazebo" />
-  <xacro:include filename="$(find bioscara_description)/urdf/bioscara.urdf.xacro" />
+  <xacro:include filename="$(find bioscara_description)/urdf/bioscara.ros2control" />
+  <xacro:bioscara_ros2_control prefix="$(arg prefix)" parameters="${params}" use_mock_hardware="$(arg use_mock_hardware)"/>
+  <!-- Used for fixing robot -->
+  <link name="world"/>
+  <xacro:bioscara parent="world" prefix="$(arg prefix)" parameters="${params}">
+    <origin xyz="0 0 0" rpy="0 0 0" />
+  </xacro:bioscara>
 </robot>

Commit message: wip: gripper

File: ROS2/ros2_scara_ws/src/dalsa_bioscara/bioscara_description/urdf/bioscara.urdf.xacro (robot description, xacro)
@@ -138,8 +138,8 @@
       <origin xyz="0 0 0" rpy="${pi} 0 0" />
       <parent link="${prefix}link_4"/>
-      <child link="${prefix}tool0" />
+      <child link="${prefix}tool_flange" />
     </joint>
     <!-- Tool Link -->
-    <link name="${prefix}tool0"/>
+    <link name="${prefix}tool_flange"/>
   </xacro:macro>
 </robot>

File: ROS2/ros2_scara_ws/src/dalsa_bioscara/bioscara_description/urdf/bioscara.xacro (robot description, xacro)
@@ -4,4 +4,20 @@
   <xacro:arg name="command_interface" default="position"/>
   <xacro:arg name="prefix" default=""/>
+  <xacro:arg name="gripper_package_name" default="" />
+  <xacro:arg name="gripper_macro_path" default="/urdf/gripper.xacro" />
+  <xacro:include filename="$(find bioscara_description)/urdf/bioscara_robot.xacro" />
+  <!-- Used for fixing robot -->
+  <link name="world"/>
+  <!-- Include the robot macro which assembles the arm and the gripper -->
+  <xacro:load_robot
+    parent="world"
+    prefix="$(arg prefix)"
+    use_mock_hardware="$(arg use_mock_hardware)"
+    command_interface="$(arg command_interface)"
+    gripper_package_name="$(arg gripper_package_name)"
+    gripper_macro_path="$(arg gripper_macro_path)">
+    <origin xyz="0 0 0" rpy="0 0 0" />
+  </xacro:load_robot>
+<!--
   <xacro:property name="config_file" value="$(find bioscara_description)/config/bioscara_parameters.yaml" />
   <xacro:property name="params" value="${xacro.load_yaml(config_file)}"/>
@@ -11,8 +27,4 @@
   <xacro:include filename="$(find bioscara_description)/urdf/bioscara.ros2control" />
   <xacro:bioscara_ros2_control prefix="$(arg prefix)" parameters="${params}" use_mock_hardware="$(arg use_mock_hardware)" command_interface="$(arg command_interface)"/>
-  <!-- Used for fixing robot -->
-  <link name="world"/>
-  <xacro:bioscara parent="world" prefix="$(arg prefix)" parameters="${params}">
-    <origin xyz="0 0 0" rpy="0 0 0" />
-  </xacro:bioscara>
+   -->
 </robot>

Commit message: change from offset to min/max

File: ROS2/ros2_scara_ws/src/dalsa_bioscara/bioscara_description/urdf/bioscara.urdf.xacro (robot description, xacro)
@@ -32,5 +32,5 @@
       <child link="${prefix}link_1"/>
       <axis xyz="0.0 0.0 1.0"/>
-      <limit upper="${fabs(parameters['j1']['offset'])}" lower="${0-fabs(parameters['j1']['offset'])}" effort="100" velocity="${parameters['j1']['max_velocity']}"/>
+      <limit upper="${parameters['j1']['max']}" lower="${parameters['j1']['min']}" effort="100" velocity="${parameters['j1']['max_velocity']}"/>
     </joint>
     <link name="${prefix}link_1">
@@ -59,5 +59,5 @@
       <child link="${prefix}link_2"/>
       <axis xyz="0.0 0.0 1.0"/>
-      <limit upper="${parameters['j2']['offset']}" lower="0" effort="100" velocity="${parameters['j2']['max_velocity']}"/>
+      <limit upper="${parameters['j2']['max']}" lower="0" effort="100" velocity="${parameters['j2']['max_velocity']}"/>
     </joint>
     <link name="${prefix}link_2">
@@ -86,5 +86,5 @@
       <child link="${prefix}link_3"/>
       <axis xyz="0.0 0.0 1.0"/>
-      <limit upper="${fabs(parameters['j3']['offset'])}" lower="${0-fabs(parameters['j3']['offset'])}" effort="100" velocity="${parameters['j3']['max_velocity']}"/>
+      <limit upper="${parameters['j3']['max']}" lower="${parameters['j3']['min']}" effort="100" velocity="${parameters['j3']['max_velocity']}"/>
     </joint>
     <link name="${prefix}link_3">
@@ -113,5 +113,5 @@
       <child link="${prefix}link_4"/>
       <axis xyz="0.0 0.0 1.0"/>
-      <limit upper="${fabs(parameters['j4']['offset'])}" lower="${0-fabs(parameters['j4']['offset'])}" effort="100" velocity="${parameters['j4']['max_velocity']}"/>
+      <limit upper="${parameters['j4']['max']}" lower="${parameters['j4']['min']}" effort="100" velocity="${parameters['j4']['max_velocity']}"/>
     </joint>
     <link name="${prefix}link_4">

Commit message: wip: restructure gripper

File: ROS2/ros2_scara_ws/src/dalsa_bioscara/bioscara_description/urdf/bioscara.urdf.xacro (robot description, xacro)
@@ -135,5 +135,5 @@
       </collision>
     </link>
-    <joint name="${prefix}tool_joint" type="fixed">
+    <joint name="${prefix}flange_joint" type="fixed">
       <origin xyz="0 0 0" rpy="${pi} 0 0" />
       <parent link="${prefix}link_4"/>

File: ROS2/ros2_scara_ws/src/dalsa_bioscara/bioscara_description/urdf/bioscara_arm.xacro (robot description, xacro)
@@ -5,5 +5,4 @@
     *origin
     use_mock_hardware
-    command_interface
     prefix">
     <xacro:property name="config_file" value="$(find bioscara_description)/config/bioscara_parameters.yaml" />
@@ -15,6 +14,5 @@
       prefix="${prefix}"
       parameters="${params}"
-      use_mock_hardware="${use_mock_hardware}"
-      command_interface="${command_interface}"/>
+      use_mock_hardware="${use_mock_hardware}"/>
     <xacro:bioscara
       parent="${parent}"

File: ROS2/ros2_scara_ws/src/dalsa_grippers/bioscara_gripper_descriptions/urdf/bioscara_gripper_128.urdf.xacro (robot description, xacro)
@@ -1,16 +1,35 @@
 <?xml version="1.0"?>
 <robot xmlns:xacro="http://wiki.ros.org/xacro" name="bioscara_gripper">
-    <xacro:macro name="bioscara_wide_gripper" params="
-        name
+    <xacro:macro name="bioscara_gripper_128" params="
+        parameters
         prefix
         parent
-        *origin
-        use_mock_hardware
-        gripper_speed_multiplier:=1.0
-        gripper_force_multiplier:=0.5
-        gripper_max_speed:=0.150
-        gripper_max_force:=235.0
-        gripper_closed_position:=0.7929">
-        <link name="${prefix}robotiq_85_base_link">
+        *origin">
+    <joint name="${prefix}base_joint" type="fixed">
+      <xacro:insert_block name="origin" />
+      <parent link="${parent}" />
+      <child link="${prefix}base_link" />
+    </joint>
+    <link name="${prefix}base_link">
+      <inertial>
+        <origin xyz="-0.04726295478480471 -4.0726333219249673e-17 0.039609285941398516" rpy="0 0 0"/>
+        <mass value="42.07322100213777"/>
+        <inertia ixx="0.19661" iyy="0.332522" izz="0.481291" ixy="-0.0" iyz="-0.0" ixz="-0.016821"/>
+      </inertial>
+      <visual>
+        <origin xyz="0 0 0" rpy="0 0 0"/>
+        <geometry>
+          <box size="0.6 0.1 0.2"/>
+        </geometry>
+        <!-- <material name="silver"/> -->
+      </visual>
+      <collision>
+        <origin xyz="0 0 0" rpy="0 0 0"/>
+        <geometry>
+          <box size="0.6 0.1 0.2"/>
+        </geometry>
+      </collision>
+    </link>
+        <!-- <link name="${prefix}robotiq_85_base_link">
             <visual>
                 <geometry>
@@ -258,5 +277,5 @@
             <origin xyz="-0.00563134 0.0 0.04718515" rpy="0 0 0" />
             <mimic joint="${prefix}robotiq_85_left_knuckle_joint" />
-        </joint>
+        </joint> -->
     </xacro:macro>
 </robot>

File: ROS2/ros2_scara_ws/src/scene_descriptions/urdf/robot.xacro (robot description, xacro)
@@ -1,21 +1,23 @@
 <?xml version="1.0" ?>
-<robot name="bioscara" xmlns:xacro="http://www.ros.org/wiki/xacro">
+<robot name="" xmlns:xacro="http://www.ros.org/wiki/xacro">
   <xacro:macro name="load_robot" params="
     parent
     *origin
     use_mock_hardware
-    command_interface
     prefix
-    gripper_package_name
+    arm_description_package
+    arm_macro_path
+    gripper_description_package
     gripper_macro_path">
+    <!-- Include and load arm macro files -->
+    <xacro:include filename="$(find ${arm_description_package})${arm_macro_path}"/>
     <xacro:load_arm
       parent="${parent}"
       prefix="${prefix}"
-      use_mock_hardware="${use_mock_hardware}"
-      command_interface="${command_interface}">
+      use_mock_hardware="${use_mock_hardware}">
       <xacro:insert_block name="origin" />
     </xacro:load_arm>
     <!-- If no gripper, define tool frame here. The last arm link must be "tool_flange" -->
-    <xacro:if value="${not gripper_package_name}">
+    <xacro:if value="${not gripper_description_package}">
       <link name="${prefix}tool"/>
       <joint name="${prefix}tool_joint" type="fixed">
@@ -27,11 +29,13 @@
     </xacro:if>
     <!-- Include and load the gripper if defined -->
-    <xacro:unless value="${not gripper_package_name}">
-    <!-- TODO: Check if the include works without "$(find <package>)" -->
-      <xacro:include filename="package://${gripper_package_name}${gripper_macro_path}"/>
+    <xacro:unless value="${not gripper_description_package}">
+      <xacro:include filename="$(find ${gripper_description_package})${gripper_macro_path}"/>
       <xacro:load_gripper
         parent="${prefix}tool_flange"
         prefix="${prefix}"
-        use_mock_hardware="${use_mock_hardware}"/>
+        use_mock_hardware="${use_mock_hardware}">
+        <!-- TODO. define origin of gripper -->
+        <origin xyz="0 0 0" rpy="0 0 0" />
+       </xacro:load_gripper>
     </xacro:unless>
   </xacro:macro>
