Commit message: feat: package launch files

File: ROS2/ros2_scara_ws/src/dalsa_bioscara/bioscara_description/urdf/bioscara.urdf.xacro (robot description, xacro)
@@ -2,4 +2,5 @@
 <robot xmlns:xacro="http://www.ros.org/wiki/xacro">
   <xacro:macro name="bioscara" params="parameters prefix parent *origin">
+    <xacro:include filename="$(find bioscara_description)/urdf/materials.xacro" />
     <joint name="${prefix}base_joint" type="fixed">
       <xacro:insert_block name="origin" />

File: ROS2/ros2_scara_ws/src/dalsa_bioscara/bioscara_description/urdf/bioscara_arm.xacro (robot description, xacro)
@@ -8,5 +8,4 @@
     <xacro:property name="config_file" value="$(find bioscara_description)/config/bioscara_parameters.yaml" />
     <xacro:property name="params" value="${xacro.load_yaml(config_file)}"/>
-    <xacro:include filename="$(find bioscara_description)/urdf/materials.xacro" />
     <xacro:include filename="$(find bioscara_description)/urdf/bioscara.urdf.xacro" />
     <xacro:include filename="$(find bioscara_description)/urdf/bioscara.ros2control" />

File: ROS2/ros2_scara_ws/src/scene_descriptions/urdf/robot.xacro (robot description, xacro)
@@ -35,6 +35,5 @@
         prefix="${prefix}"
         use_mock_hardware="${use_mock_hardware}">
-        <!-- TODO. define origin of gripper -->
-        <origin xyz="0 0 0" rpy="0 0 0" />
+        <origin xyz="0 0 0" rpy="${pi} 0 ${-pi/2}" />
        </xacro:load_gripper>
     </xacro:unless>

File: ROS2/ros2_scara_ws/src/scene_descriptions/urdf/scene.xacro (robot description, xacro)
@@ -1,6 +1,5 @@
 <?xml version="1.0" ?>
-<robot name="bioscara" xmlns:xacro="http://www.ros.org/wiki/xacro">
+<robot name="scene" xmlns:xacro="http://www.ros.org/wiki/xacro">
   <xacro:arg name="use_mock_hardware" default="false"/>
-  <!-- <xacro:arg name="prefix" default=""/> Does it make sense to have a prefix for a scene? -->
   <xacro:arg name="arm_description_package" default="bioscara_description" />
   <xacro:arg name="arm_macro_path" default="/urdf/bioscara_arm.xacro" />
