Commit message: feat: complete launch files in bringup and description packages

File: ROS2/ros2_scara_ws/src/dalsa_bioscara/bioscara_description/urdf/scene.xacro (robot description, xacro)
@@ -3,10 +3,10 @@
   <xacro:arg name="use_mock_hardware" default="false"/>
   <xacro:arg name="prefix" default=""/>
-  <xacro:arg name="arm_macro_path" default="/urdf/bioscara_arm.xacro" />
+  <xacro:arg name="arm_macro" default="bioscara_arm.xacro" />
   <xacro:property name="arm_description_package" value="$(arg arm_description_package)"/>
-  <xacro:property name="arm_macro_path" value="$(arg arm_macro_path)"/>
+  <xacro:property name="arm_macro" value="$(arg arm_macro)"/>
   <!-- Used for fixing robot -->
   <link name="world"/>
-  <xacro:include filename="$(find bioscara_description)${arm_macro_path}"/>
+  <xacro:include filename="$(find bioscara_description)/urdf/${arm_macro}"/>
   <xacro:load_arm
     parent="world"

File: ROS2/ros2_scara_ws/src/dalsa_grippers/bioscara_gripper_descriptions/urdf/scene.xacro (robot description, xacro)
@@ -3,7 +3,7 @@
   <xacro:arg name="use_mock_hardware" default="false"/>
   <xacro:arg name="prefix" default=""/>
-  <xacro:arg name="gripper_macro_path" default="/urdf/bioscara_gripper_128.xacro" />
-  <xacro:property name="gripper_macro_path" value="$(arg gripper_macro_path)"/>
-  <xacro:include filename="$(find bioscara_gripper_descriptions)${gripper_macro_path}"/>
+  <xacro:arg name="gripper_macro" default="bioscara_gripper_128.xacro" />
+  <xacro:property name="gripper_macro" value="$(arg gripper_macro)"/>
+  <xacro:include filename="$(find bioscara_gripper_descriptions)/urdf/${gripper_macro}"/>
   <!-- Used for fixing robot -->
   <link name="world"/>

File: ROS2/ros2_scara_ws/src/scene_descriptions/urdf/robot.xacro (robot description, xacro)
@@ -7,9 +7,9 @@
     prefix
     arm_description_package
-    arm_macro_path
+    arm_macro
     gripper_description_package
-    gripper_macro_path">
+    gripper_macro">
     <!-- Include and load arm macro files -->
-    <xacro:include filename="$(find ${arm_description_package})${arm_macro_path}"/>
+    <xacro:include filename="$(find ${arm_description_package})/urdf/${arm_macro}"/>
     <xacro:load_arm
       parent="${parent}"
@@ -30,5 +30,5 @@
     <!-- Include and load the gripper if defined -->
     <xacro:unless value="${not gripper_description_package}">
-      <xacro:include filename="$(find ${gripper_description_package})${gripper_macro_path}"/>
+      <xacro:include filename="$(find ${gripper_description_package})/urdf/${gripper_macro}"/>
       <xacro:load_gripper
         parent="${prefix}tool_flange"

File: ROS2/ros2_scara_ws/src/scene_descriptions/urdf/scene.xacro (robot description, xacro)
@@ -3,7 +3,7 @@
   <xacro:arg name="use_mock_hardware" default="false"/>
   <xacro:arg name="arm_description_package" default="bioscara_description" />
-  <xacro:arg name="arm_macro_path" default="/urdf/bioscara_arm.xacro" />
+  <xacro:arg name="arm_macro" default="bioscara_arm.xacro" />
   <xacro:arg name="gripper_description_package" default="" />
-  <xacro:arg name="gripper_macro_path" default="/urdf/bioscara_gripper_128.xacro" />
+  <xacro:arg name="gripper_macro" default="bioscara_gripper_128.xacro" />
   <xacro:include filename="$(find scene_descriptions)/urdf/robot.xacro" />
   <!-- Used for fixing robot -->
@@ -15,7 +15,7 @@
     use_mock_hardware="$(arg use_mock_hardware)"
     arm_description_package="$(arg arm_description_package)"
-    arm_macro_path="$(arg arm_macro_path)"
+    arm_macro="$(arg arm_macro)"
     gripper_description_package="$(arg gripper_description_package)"
-    gripper_macro_path="$(arg gripper_macro_path)">
+    gripper_macro="$(arg gripper_macro)">
     <origin xyz="0 0 0" rpy="0 0 0" />
   </xacro:load_robot>
