Commit message: feat: gripper HW IF works

File: ROS2/ros2_scara_ws/src/dalsa_grippers/bioscara_gripper_descriptions/urdf/bioscara_gripper_128.ros2_control.xacro (robot description, xacro)
@@ -16,49 +16,11 @@
             </hardware>
             <!-- Joint interfaces -->
-            <!-- With Gazebo or Hardware, they handle mimic joints, so we only need this command interface activated -->
-            <joint name="${prefix}left_jaw">
+            <joint name="${prefix}gripper">
                 <command_interface name="position" />
                 <state_interface name="position"/>
+                <!-- Does not actually have a sensor, is emulated as derivative of position.
+                Is needed for GripperActionController. -->
+                <state_interface name="velocity"/>
             </joint>
-            <!-- When simulating we need to include the rest of the gripper joints -->
-            <!-- <xacro:if value="${use_mock_hardware or sim_isaac or sim_gazebo}">
-                <joint name="${prefix}robotiq_85_right_knuckle_joint">
-                    <xacro:unless value="${sim_gazebo}">
-                        <state_interface name="position"/>
-                        <state_interface name="velocity"/>
-                    </xacro:unless>
-                </joint>
-                <joint name="${prefix}robotiq_85_left_inner_knuckle_joint">
-                    <xacro:unless value="${sim_gazebo}">
-                        <state_interface name="position"/>
-                        <state_interface name="velocity"/>
-                    </xacro:unless>
-                </joint>
-                <joint name="${prefix}robotiq_85_right_inner_knuckle_joint">
-                    <xacro:unless value="${sim_gazebo}">
-                        <state_interface name="position"/>
-                        <state_interface name="velocity"/>
-                    </xacro:unless>
-                </joint>
-                <joint name="${prefix}robotiq_85_left_finger_tip_joint">
-                    <xacro:unless value="${sim_gazebo}">
-                        <state_interface name="position"/>
-                        <state_interface name="velocity"/>
-                    </xacro:unless>
-                </joint>
-                <joint name="${prefix}robotiq_85_right_finger_tip_joint">
-                    <xacro:unless value="${sim_gazebo}">
-                        <state_interface name="position"/>
-                        <state_interface name="velocity"/>
-                    </xacro:unless>
-                </joint>
-            </xacro:if> -->
-            <!-- Only add this with fake hardware mode -->
-            <!-- <xacro:unless value="${sim_gazebo or sim_isaac}">
-                <gpio name="reactivate_gripper">
-                    <command_interface name="reactivate_gripper_cmd" />
-                    <command_interface name="reactivate_gripper_response" />
-                </gpio>
-            </xacro:unless> -->
         </ros2_control>
     </xacro:macro>

File: ROS2/ros2_scara_ws/src/dalsa_grippers/bioscara_gripper_descriptions/urdf/bioscara_gripper_128.urdf.xacro (robot description, xacro)
@@ -6,276 +6,79 @@
         parent
         *origin">
-    <joint name="${prefix}base_joint" type="fixed">
-      <xacro:insert_block name="origin" />
-      <parent link="${parent}" />
-      <child link="${prefix}base_link" />
-    </joint>
-    <link name="${prefix}base_link">
-      <inertial>
-        <origin xyz="-0.04726295478480471 -4.0726333219249673e-17 0.039609285941398516" rpy="0 0 0"/>
-        <mass value="42.07322100213777"/>
-        <inertia ixx="0.19661" iyy="0.332522" izz="0.481291" ixy="-0.0" iyz="-0.0" ixz="-0.016821"/>
-      </inertial>
-      <visual>
-        <origin xyz="0 0 0" rpy="0 0 0"/>
-        <geometry>
-          <box size="0.6 0.1 0.2"/>
-        </geometry>
-        <!-- <material name="silver"/> -->
-      </visual>
-      <collision>
-        <origin xyz="0 0 0" rpy="0 0 0"/>
-        <geometry>
-          <box size="0.6 0.1 0.2"/>
-        </geometry>
-      </collision>
-    </link>
-        <!-- <link name="${prefix}robotiq_85_base_link">
+        <xacro:include filename="$(find bioscara_gripper_descriptions)/urdf/materials.xacro" />
+        <joint name="${prefix}grp_base_joint" type="fixed">
+            <xacro:insert_block name="origin" />
+            <parent link="${parent}" />
+            <child link="${prefix}grp_base_link" />
+        </joint>
+        <link name="${prefix}grp_base_link">
+            <visual>
+                <origin xyz="0 0 0" rpy="0 0 0"/>
+                <geometry>
+                    <mesh filename="file://$(find bioscara_gripper_descriptions)/meshes/base.stl" scale="0.001 0.001 0.001"/>
+                </geometry>
+                <material name="gripper_silver"/>
+            </visual>
+            <collision>
+                <origin xyz="0 0 0" rpy="0 0 0"/>
+                <geometry>
+                    <mesh filename="file://$(find bioscara_gripper_descriptions)/meshes/base.stl" scale="0.001 0.001 0.001"/>
+                </geometry>
+            </collision>
+        </link>
+        <link name="${prefix}virtual_gripper"/>
+        <joint name="${prefix}gripper" type="prismatic">
+            <parent link="${prefix}grp_base_link"/>
+            <child link="${prefix}virtual_gripper"/>
+            <axis xyz="1.0 0.0 0.0"/>
+            <limit upper="${parameters['max']}" lower="${parameters['min']}" effort="100" velocity="${parameters['max_velocity']}"/>
+        </joint>
+        <link name="${prefix}left_jaw_link">
             <visual>
                 <geometry>
-                    <mesh filename="package://robotiq_description/meshes/visual/2f_85/robotiq_base.dae" />
+                    <mesh filename="file://$(find bioscara_gripper_descriptions)/meshes/left_jaw.stl" scale="0.001 0.001 0.001"/>
                 </geometry>
+                <material name="gripper_silver"/>
             </visual>
             <collision>
                 <geometry>
-                    <mesh filename="package://robotiq_description/meshes/collision/2f_85/robotiq_base.stl" />
+                    <mesh filename="file://$(find bioscara_gripper_descriptions)/meshes/left_jaw.stl" scale="0.001 0.001 0.001"/>
                 </geometry>
             </collision>
-            <inertial>
-                <origin xyz="0.0 2.274e-05 0.03232288" rpy="0 0 0" />
-                <mass value="6.6320197e-01" />
-                <inertia ixx="5.1617816e-04" iyy="5.8802208e-04" izz="3.9462776e-04" ixy="2.936e-8" ixz="0.0" iyz="-3.2296e-7" />
-            </inertial>
         </link>
-        <link name="${prefix}robotiq_85_left_knuckle_link">
+        <link name="${prefix}right_jaw_link">
             <visual>
                 <geometry>
-                    <mesh filename="package://robotiq_description/meshes/visual/2f_85/left_knuckle.dae" />
+                    <mesh filename="file://$(find bioscara_gripper_descriptions)/meshes/right_jaw.stl" scale="0.001 0.001 0.001"/>
                 </geometry>
+                <material name="gripper_silver"/>
             </visual>
             <collision>
                 <geometry>
-                    <mesh filename="package://robotiq_description/meshes/collision/2f_85/left_knuckle.stl" />
+                    <mesh filename="file://$(find bioscara_gripper_descriptions)/meshes/right_jaw.stl" scale="0.001 0.001 0.001"/>
                 </geometry>
             </collision>
-            <inertial>
-                <origin xyz="0.01213197 0.0002 -0.00058647" rpy="0 0 0" />
-                <mass value="1.384773208e-02" />
-                <inertia ixx="3.5232e-7" iyy="2.31944e-6" izz="2.23136e-6" ixy="0.0" ixz="1.1744e-7" iyz="0" />
-            </inertial>
         </link>
-        <link name="${prefix}robotiq_85_right_knuckle_link">
-            <visual>
-                <geometry>
-                    <mesh filename="package://robotiq_description/meshes/visual/2f_85/right_knuckle.dae" />
-                </geometry>
-            </visual>
-            <collision>
-                <geometry>
-                    <mesh filename="package://robotiq_description/meshes/collision/2f_85/right_knuckle.stl" />
-                </geometry>
-            </collision>
-            <inertial>
-                <origin xyz="-0.01213197 0.0002 -0.00058647" rpy="0 0 0" />
-                <mass value="1.384773208e-02" />
-                <inertia ixx="3.5232e-7" iyy="2.31944e-6" izz="2.23136e-6" ixy="0.0" ixz="-1.1744e-7" iyz="0.0" />
-            </inertial>
-        </link>
-        <link name="${prefix}robotiq_85_left_finger_link">
-            <visual>
-                <geometry>
-                    <mesh filename="package://robotiq_description/meshes/visual/2f_85/left_finger.dae" />
-                </geometry>
-            </visual>
-            <collision>
-                <geometry>
-                    <mesh filename="package://robotiq_description/meshes/collision/2f_85/left_finger.stl" />
-                </geometry>
-            </collision>
-            <inertial>
-                <origin xyz="0.00346899 -0.00079447 0.01867121" rpy="0 0 0" />
-                <mass value="4.260376752e-02" />
-                <inertia ixx="1.385792000000000e-05" iyy="1.183208e-05" izz="5.19672e-06" ixy="0.0" ixz="-2.17264e-06" iyz="0.0" />
-            </inertial>
-        </link>
-        <link name="${prefix}robotiq_85_right_finger_link">
-            <visual>
-                <geometry>
-                    <mesh filename="package://robotiq_description/meshes/visual/2f_85/right_finger.dae" />
-                </geometry>
-            </visual>
-            <collision>
-                <geometry>
-                    <mesh filename="package://robotiq_description/meshes/collision/2f_85/right_finger.stl" />
-                </geometry>
-            </collision>
-            <inertial>
-                <origin xyz="-0.00346899 -5.53e-06 0.01867121" rpy="0 0 0" />
-                <mass value="4.260376752000000e-02" />
-                <inertia ixx="1.385792e-05" iyy="1.183208e-05" izz="5.19672e-06" ixy="0.0" ixz="2.17264e-06" iyz="0.0" />
-            </inertial>
-        </link>
-        <link name="${prefix}robotiq_85_left_inner_knuckle_link">
-            <visual>
-                <geometry>
-                    <mesh filename="package://robotiq_description/meshes/visual/2f_85/left_inner_knuckle.dae" />
-                </geometry>
-            </visual>
-            <collision>
-                <geometry>
-                    <mesh filename="package://robotiq_description/meshes/collision/2f_85/left_inner_knuckle.stl" />
-                </geometry>
-            </collision>
-            <inertial>
-                <origin xyz="0.01897699 0.00015001 0.02247101" rpy="0 0 0" />
-                <mass value="2.969376448e-02" />
-                <inertia ixx="9.57136e-06" iyy="8.69056e-06" izz="8.19144e-06" ixy="0.0" ixz="-3.93424e-06" iyz="0.0" />
-            </inertial>
-        </link>
-        <link name="${prefix}robotiq_85_right_inner_knuckle_link">
-            <visual>
-                <geometry>
-                    <mesh filename="package://robotiq_description/meshes/visual/2f_85/right_inner_knuckle.dae" />
-                </geometry>
-            </visual>
-            <collision>
-                <geometry>
-                    <mesh filename="package://robotiq_description/meshes/collision/2f_85/right_inner_knuckle.stl" />
-                </geometry>
-            </collision>
-            <inertial>
-                <origin xyz="-0.01926824 5.001e-05 0.02222178" rpy="0 0 0" />
-                <mass value="2.969376448e-02" />
-                <inertia ixx="9.42456e-06" iyy="8.69056e-06" izz="8.33824e-06" ixy="0.0" ixz="3.9636e-06" iyz="0.0" />
-            </inertial>
-        </link>
-        <link name="${prefix}robotiq_85_left_finger_tip_link">
-            <visual>
-                <geometry>
-                    <mesh filename="package://robotiq_description/meshes/visual/2f_85/left_finger_tip.dae" />
-                </geometry>
-            </visual>
-            <collision>
-                <geometry>
-                    <mesh filename="package://robotiq_description/meshes/collision/2f_85/left_finger_tip.stl" />
-                </geometry>
-                <surface>
-                    <friction>
-                    <ode>
-                        <mu1>100000.0</mu1>
-                        <mu2>100000.0</mu2>
-                    </ode>
-                    </friction>
-                    <contact>
-                    <ode>
-                        <kp>1e+5</kp>
-                        <kd>1</kd>
-                        <soft_cfm>0</soft_cfm>
-                        <soft_erp>0.2</soft_erp>
-                        <minDepth>0.002</minDepth>
-                        <maxVel>0</maxVel>
-                    </ode>
-                    </contact>
-                </surface>
-            </collision>
-            <inertial>
-                <origin xyz="-0.01456706 -0.0008 0.01649701" rpy="0 0 0" />
-                <mass value="4.268588744e-02" />
-                <inertia ixx="1.048152e-05" iyy="1.197888e-05" izz="4.22784e-06" ixy="0.0" ixz="3.5232e-6" iyz="0.0" />
-            </inertial>
-        </link>
-        <link name="${prefix}robotiq_85_right_finger_tip_link">
-            <visual>
-                <geometry>
-                    <mesh filename="package://robotiq_description/meshes/visual/2f_85/right_finger_tip.dae" />
-                </geometry>
-            </visual>
-            <collision>
-                <geometry>
-                    <mesh filename="package://robotiq_description/meshes/collision/2f_85/right_finger_tip.stl" />
-                </geometry>
-                <surface>
-                    <friction>
-                    <ode>
-                        <mu1>100000.0</mu1>
-                        <mu2>100000.0</mu2>
-                    </ode>
-                    </friction>
-                    <contact>
-                    <ode>
-                        <kp>1e+5</kp>
-                        <kd>1</kd>
-                        <soft_cfm>0</soft_cfm>
-                        <soft_erp>0.2</soft_erp>
-                        <minDepth>0.002</minDepth>
-                        <maxVel>0</maxVel>
-                    </ode>
-                    </contact>
-                </surface>
-            </collision>
-            <inertial>
-                <origin xyz="0.01456706 5e-05 0.01649701" rpy="0 0 0" />
-                <mass value="4.268588744e-02" />
-                <inertia ixx="1.048152e-05" iyy="1.197888e-05" izz="4.22784e-06" ixy="0.0" ixz="-3.5232e-06" iyz="0.0" />
-            </inertial>
-        </link>
-        <joint name="${prefix}robotiq_85_base_joint" type="fixed">
-            <parent link="${parent}" />
-            <child link="${prefix}robotiq_85_base_link" />
-            <xacro:insert_block name="origin" />
+        <joint name="${prefix}gripper_l_mimic" type="prismatic">
+            <parent link="${prefix}grp_base_link"/>
+            <child link="${prefix}left_jaw_link"/>
+            <axis xyz="1 0 0" />
+            <limit upper="${parameters['max']}" lower="${parameters['min']}" effort="100" velocity="${parameters['max_velocity']}"/>
+            <mimic joint="${prefix}gripper" multiplier="0.5" />
         </joint>
-        <joint name="${prefix}robotiq_85_left_knuckle_joint" type="revolute">
-            <parent link="${prefix}robotiq_85_base_link" />
-            <child link="${prefix}robotiq_85_left_knuckle_link" />
-            <axis xyz="0 -1 0" />
-            <origin xyz="0.03060114 0.0 0.05490452" rpy="0 0 0" />
-            <limit lower="0.0" upper="0.8" velocity="0.5" effort="50" />
+        <joint name="${prefix}gripper_r_mimic" type="prismatic">
+            <parent link="${prefix}grp_base_link"/>
+            <child link="${prefix}right_jaw_link"/>
+            <axis xyz="1 0 0" />
+            <limit upper="${parameters['max']}" lower="${parameters['min']}" effort="100" velocity="${parameters['max_velocity']}"/>
+            <mimic joint="${prefix}gripper" multiplier="-0.5" />
         </joint>
-        <joint name="${prefix}robotiq_85_right_knuckle_joint" type="revolute">
-            <parent link="${prefix}robotiq_85_base_link" />
-            <child link="${prefix}robotiq_85_right_knuckle_link" />
-            <axis xyz="0 -1 0" />
-            <origin xyz="-0.03060114 0.0 0.05490452" rpy="0 0 0" />
-            <limit lower="-0.8" upper="0.0" velocity="0.5" effort="50" />
-            <mimic joint="${prefix}robotiq_85_left_knuckle_joint" multiplier="-1" />
+        <!-- Tool Link -->
+        <link name="${prefix}tool"/>
+        <joint name="tool" type="fixed">
+            <parent link="${prefix}grp_base_link"/>
+            <child link="${prefix}tool"/>
+            <origin xyz="0.0 -0.11908 -0.14409" rpy="0 0 ${-pi/2}" />
         </joint>
-        <joint name="${prefix}robotiq_85_left_finger_joint" type="fixed">
-            <parent link="${prefix}robotiq_85_left_knuckle_link" />
-            <child link="${prefix}robotiq_85_left_finger_link" />
-            <origin xyz="0.03152616 0.0 -0.00376347" rpy="0 0 0" />
-        </joint>
-        <joint name="${prefix}robotiq_85_right_finger_joint" type="fixed">
-            <parent link="${prefix}robotiq_85_right_knuckle_link" />
-            <child link="${prefix}robotiq_85_right_finger_link" />
-            <origin xyz="-0.03152616 0.0 -0.00376347" rpy="0 0 0" />
-        </joint>
-        <joint name="${prefix}robotiq_85_left_inner_knuckle_joint" type="continuous">
-            <parent link="${prefix}robotiq_85_base_link" />
-            <child link="${prefix}robotiq_85_left_inner_knuckle_link" />
-            <axis xyz="0 -1 0" />
-            <origin xyz="0.0127 0.0 0.06142" rpy="0 0 0" />
-            <mimic joint="${prefix}robotiq_85_left_knuckle_joint" />
-        </joint>
-        <joint name="${prefix}robotiq_85_right_inner_knuckle_joint" type="continuous">
-            <parent link="${prefix}robotiq_85_base_link" />
-            <child link="${prefix}robotiq_85_right_inner_knuckle_link" />
-            <axis xyz="0 -1 0" />
-            <origin xyz="-0.0127 0.0 0.06142" rpy="0 0 0" />
-            <mimic joint="${prefix}robotiq_85_left_knuckle_joint" multiplier="-1" />
-        </joint>
-        <joint name="${prefix}robotiq_85_left_finger_tip_joint" type="continuous">
-            <parent link="${prefix}robotiq_85_left_finger_link" />
-            <child link="${prefix}robotiq_85_left_finger_tip_link" />
-            <axis xyz="0 -1 0" />
-            <origin xyz="0.00563134 0.0 0.04718515" rpy="0 0 0" />
-            <mimic joint="${prefix}robotiq_85_left_knuckle_joint" multiplier="-1" />
-        </joint>
-        <joint name="${prefix}robotiq_85_right_finger_tip_joint" type="continuous">
-            <parent link="${prefix}robotiq_85_right_finger_link" />
-            <child link="${prefix}robotiq_85_right_finger_tip_link" />
-            <axis xyz="0 -1 0" />
-            <origin xyz="-0.00563134 0.0 0.04718515" rpy="0 0 0" />
-            <mimic joint="${prefix}robotiq_85_left_knuckle_joint" />
-        </joint> -->
     </xacro:macro>
 </robot>
