Commit message: fix: mimic joint limits

File: ROS2/ros2_scara_ws/src/dalsa_grippers/bioscara_gripper_descriptions/urdf/bioscara_gripper_128.urdf.xacro (robot description, xacro)
@@ -64,5 +64,5 @@
             <child link="${prefix}left_jaw_link"/>
             <axis xyz="1 0 0" />
-            <limit upper="${parameters['max']}" lower="${parameters['min']}" effort="100" velocity="${parameters['max_velocity']}"/>
+            <limit upper="100" lower="-100" effort="100" velocity="100"/>
             <mimic joint="${prefix}gripper" multiplier="0.5" />
         </joint>
@@ -71,5 +71,5 @@
             <child link="${prefix}right_jaw_link"/>
             <axis xyz="1 0 0" />
-            <limit upper="${parameters['max']}" lower="${parameters['min']}" effort="100" velocity="${parameters['max_velocity']}"/>
+            <limit upper="100" lower="-100" effort="100" velocity="100"/>
             <mimic joint="${prefix}gripper" multiplier="-0.5" />
         </joint>
