Commit message: renames

File: ROS2/ros2_scara_ws/src/dalsa_bioscara_arm/bioscara_arm_description/urdf/bioscara_arm.xacro (robot description, xacro)
@@ -6,5 +6,5 @@
     use_mock_hardware
     prefix">
-    <xacro:property name="config_file" value="$(find bioscara_arm_description)/config/bioscara_parameters.yaml" />
+    <xacro:property name="config_file" value="$(find bioscara_arm_description)/config/bioscara_arm_parameters.yaml" />
     <xacro:property name="params" value="${xacro.load_yaml(config_file)}"/>
     <xacro:include filename="$(find bioscara_arm_description)/urdf/bioscara.urdf.xacro" />

File: ROS2/ros2_scara_ws/src/scene_descriptions/urdf/robot.xacro (robot description, xacro)
@@ -1,4 +1,4 @@
 <?xml version="1.0" ?>
-<robot name="" xmlns:xacro="http://www.ros.org/wiki/xacro">
+<robot name="robot" xmlns:xacro="http://www.ros.org/wiki/xacro">
   <xacro:macro name="load_robot" params="
     parent
