Commit message: fix: correct tool_flange z-height (#27)

File: ROS2/ros2_scara_ws/src/dalsa_bioscara_arm/bioscara_arm_description/urdf/bioscara.urdf.xacro (robot description, xacro)
@@ -3,4 +3,5 @@
   <xacro:macro name="bioscara" params="parameters prefix parent *origin">
     <xacro:include filename="$(find bioscara_arm_description)/urdf/materials.xacro" />
+    <xacro:property name="tool_flange_zheight" value="0.135"/>
     <joint name="${prefix}base_joint" type="fixed">
       <xacro:insert_block name="origin" />
@@ -29,5 +30,5 @@
     </link>
     <joint name="${prefix}j1" type="revolute">
-      <origin xyz="0.0 0.0 0.1442" rpy="0 0 0"/>
+      <origin xyz="0.0 0.0 ${tool_flange_zheight}" rpy="0 0 0"/>
       <parent link="${prefix}base_link"/>
       <child link="${prefix}link_1"/>
@@ -42,5 +43,5 @@
       </inertial>
       <visual>
-        <origin xyz="-0.0 -0.0 -0.1442" rpy="0 0 0"/>
+        <origin xyz="-0.0 -0.0 -${tool_flange_zheight}" rpy="0 0 0"/>
         <geometry>
           <mesh filename="file://$(find bioscara_arm_description)/meshes/link_1_1.stl" scale="0.001 0.001 0.001"/>
@@ -49,5 +50,5 @@
       </visual>
       <collision>
-        <origin xyz="-0.0 -0.0 -0.1442" rpy="0 0 0"/>
+        <origin xyz="-0.0 -0.0 -${tool_flange_zheight}" rpy="0 0 0"/>
         <geometry>
           <mesh filename="file://$(find bioscara_arm_description)/meshes/link_1_1.stl" scale="0.001 0.001 0.001"/>
@@ -69,5 +70,5 @@
       </inertial>
       <visual>
-        <origin xyz="-0.0 -0.0 -0.1442" rpy="0 0 0"/>
+        <origin xyz="-0.0 -0.0 -${tool_flange_zheight}" rpy="0 0 0"/>
         <geometry>
           <mesh filename="file://$(find bioscara_arm_description)/meshes/link_2_1.stl" scale="0.001 0.001 0.001"/>
@@ -76,5 +77,5 @@
       </visual>
       <collision>
-        <origin xyz="-0.0 -0.0 -0.1442" rpy="0 0 0"/>
+        <origin xyz="-0.0 -0.0 -${tool_flange_zheight}" rpy="0 0 0"/>
         <geometry>
           <mesh filename="file://$(find bioscara_arm_description)/meshes/link_2_1.stl" scale="0.001 0.001 0.001"/>
@@ -96,5 +97,5 @@
       </inertial>
       <visual>
-        <origin xyz="-0.329476 -0.0 -0.1442" rpy="0 0 0"/>
+        <origin xyz="-0.329476 -0.0 -${tool_flange_zheight}" rpy="0 0 0"/>
         <geometry>
           <mesh filename="file://$(find bioscara_arm_description)/meshes/link_3_1.stl" scale="0.001 0.001 0.001"/>
@@ -103,5 +104,5 @@
       </visual>
       <collision>
-        <origin xyz="-0.329476 -0.0 -0.1442" rpy="0 0 0"/>
+        <origin xyz="-0.329476 -0.0 -${tool_flange_zheight}" rpy="0 0 0"/>
         <geometry>
           <mesh filename="file://$(find bioscara_arm_description)/meshes/link_3_1.stl" scale="0.001 0.001 0.001"/>
@@ -123,5 +124,5 @@
       </inertial>
       <visual>
-        <origin xyz="-0.614476 0.0 -0.1442" rpy="0 0 0"/>
+        <origin xyz="-0.614476 0.0 -${tool_flange_zheight}" rpy="0 0 0"/>
         <geometry>
           <mesh filename="file://$(find bioscara_arm_description)/meshes/link_4_1.stl" scale="0.001 0.001 0.001"/>
@@ -130,5 +131,5 @@
       </visual>
       <collision>
-        <origin xyz="-0.614476 0.0 -0.1442" rpy="0 0 0"/>
+        <origin xyz="-0.614476 0.0 -${tool_flange_zheight}" rpy="0 0 0"/>
         <geometry>
           <mesh filename="file://$(find bioscara_arm_description)/meshes/link_4_1.stl" scale="0.001 0.001 0.001"/>
